File: hardware/pcb/FreedomWing.sch (EAGLE design)
At the start: 12 parts

Commit message: First changes after Launch
Updated to add Schottky Diodes, Reset Switch & Jumper
Parts:
- removed SJ1: (no value), jumper:SJW
- added D1, D2: (no value), adafruit:SCHOTTKY-DIODEDO41-7
- added RESET: 1825966-1, ATMakers:1825966-1
- added USB, VBAT: (no value), jumper:SJW
Connections:
- removed net N$28: JP1.1, MS1.!RESET
- removed net N$8: J2.5, SJ1.1
- new net RESET: JP1.1, MS1.!RESET, RESET.1
- new net VMAX: D1.C, D2.C, POLOLU.1, USB.1, VBAT.1
- net GND: now also RESET.2
- net N$4: no longer SJ1.2
- net USB: now also D1.A, USB.2; no longer POLOLU.1
- net VBAT: now also D2.A, VBAT.2
